Commit message: ok visual and crash

File: rod_bvp_gazebo/launch/joint.sdf.xacro (robot description, xacro)
@@ -41,6 +41,5 @@
         </inertial>
     </link>
-    <joint name="rev_joint" type="revolute">
-        <axis xyz="0 0 1"/>
+    <joint name="rev_joint" type="fixed">
         <origin xyz="0 0 0" rpy="0 0 0"/>
         <parent>base_link</parent>
