Commit message: developed plugin

File: dual_links_robot_gazebo/launch/distal_plate.sdf.xacro (robot description, xacro)
@@ -8,5 +8,21 @@
     <xacro:property name="y" value=".1"/>
     <xacro:property name="z" value=".1"/>
-    <link name="base_link2"/>
+    <xacro:arg name="enable_physics_plugin" default="true"/>
+    <xacro:arg name="fxy" default="10"/>
+    <xacro:arg name="fz" default="50"/>
+    <xacro:arg name="mz" default="0.1"/>
+    <xacro:arg name="damping" default="0.1"/>
+    <xacro:arg name="length" default="1"/>
+<!-- Model plugin for physics -->
+  <xacro:if value="$(arg enable_physics_plugin)">
+    <plugin name="dual_links_robot_physics_plugin" filename="libdual_links_robot_physics_plugin.so">
+        <fxy>$(arg fxy)</fxy>
+        <fz>$(arg fz)</fz>
+        <mz>$(arg mz)</mz>
+        <damping>$(arg damping)</damping>
+        <length>$(arg length)</length>
+        <attach_point>0 0 0</attach_point>
+    </plugin>
+  </xacro:if>
     <link name="distal_plate">
         <visual name="box">
@@ -42,9 +58,4 @@
         </inertial>
     </link>
-    <joint name="root" type="fixed">
-        <origin xyz="0 0 0" rpy="$0 0 0"/>
-        <parent>base_link2</parent>
-        <child>distal_plate</child>
-    </joint>
 </model>
 </sdf>

File: dual_links_robot_gazebo/launch/joint.sdf.xacro (robot description, xacro)
@@ -8,8 +8,10 @@
     <xacro:property name="y" value="0.05"/>
     <xacro:property name="z" value="0.1"/>
-    <xacro:arg name="joint_number"  default="0"   />
-    <link name="base_link"/>
-    <link name="joint">
-        <visual name="revolute_visual">
+    <xacro:arg name="joint_number"  default="0"/>
+    <xacro:arg name="delta_x"  default="0"/>
+    <xacro:arg name="delta_y"  default="0"/>
+    <!--<link name="base_link"/>-->
+    <link name="rev_joint$(arg joint_number)_body">
+        <visual name="rev_joint$(arg joint_number)_visual">
             <plugin name="dual_links_robot_visual_plugin" filename="libdual_links_robot_visual_plugin.so">
                 <radius>0.05</radius>
@@ -23,5 +25,5 @@
             </geometry>
         </visual>
-        <collision name="revolute_collision">
+        <collision name="rev_joint$(arg joint_number)_collision">
             <geometry>
                 <cylinder>
@@ -43,9 +45,12 @@
         </inertial>
     </link>
-    <joint name="rev_joint" type="fixed">
-        <origin xyz="0 0 0" rpy="0 0 0"/>
+    <!--<joint name="rev_joint$(arg joint_number)" type="revolute">
+        <pose>0 0 0 0 0 0</pose>
         <parent>base_link</parent>
-        <child>joint</child>
-    </joint>
+        <child>rev_joint$(arg joint_number)_body</child>
+        <axis>
+            <xyz>0 0 1</xyz>
+        </axis>
+    </joint>-->
 </model>
 </sdf>

File: dual_links_robot_gazebo/launch/joint1.sdf.xacro (robot description, xacro)
@@ -8,10 +8,13 @@
     <xacro:property name="y" value="0.05"/>
     <xacro:property name="z" value="0.1"/>
+    <xacro:arg name="joint_number"  default="1"/>
+    <xacro:arg name="delta_x"  default="0"/>
+    <xacro:arg name="delta_y"  default="0"/>
     <link name="base_link"/>
-    <link name="joint">
-        <visual name="revolute_visual">
+    <link name="rev_joint1_body">
+        <visual name="rev_joint1_visual">
             <plugin name="dual_links_robot_visual_plugin" filename="libdual_links_robot_visual_plugin.so">
                 <radius>0.05</radius>
-                <joint_number>1</joint_number>
+                <joint_number>$(arg joint_number)</joint_number>
             </plugin>
             <geometry>
@@ -22,5 +25,5 @@
             </geometry>
         </visual>
-        <collision name="revolute_collision">
+        <collision name="rev_joint1_collision">
             <geometry>
                 <cylinder>
@@ -42,8 +45,11 @@
         </inertial>
     </link>
-    <joint name="rev_joint" type="fixed">
-        <origin xyz="0 0 0" rpy="0 0 0"/>
+    <joint name="fixing" type="fixed">
+        <parent>world</parent>
+        <child>base_link</child>
+    </joint>
+    <joint name="rev_joint1" type="fixed">
         <parent>base_link</parent>
-        <child>joint</child>
+        <child>rev_joint1_body</child>
     </joint>
 </model>
